File: hardware/nRF54L15_kailh/swplate/swplate.kicad_pcb (KiCad board)
At the start: 2 copper layers, 328.1 x 198.6 mm, 102 parts

Commit message: A  hardware/nRF54L15_kailh/.gitignore M  hardware/nRF54L15_kailh/border.py A  hardware/nRF54L15_kailh/botcase/botcase-Edge_Cuts.dxf A  hardware/nRF54L15_kailh/botcase/botcase-Edge_Cuts.gm1 A  hardware/nRF54L15_kailh/botcase/botcase-Edge_Cuts.svg A  hardware/nRF54L15_kailh/botcase/botcase.kicad_pcb A  hardware/nRF54L15_kailh/botcase/botcase.kicad_prl A  hardware/nRF54L15_kailh/botcase/botcase.kicad_pro A  hardware/nRF54L15_kailh/botcase/botcase.kicad_sch A  hardware/nRF54L15_kailh/botcase/fp-lib-table A  hardware/nRF54L15_kailh/botcase/sym-lib-table A  hardware/nRF54L15_kailh/kerf.py D  hardware/nRF54L15_kailh/pat1.kicad_mod D  hardware/nRF54L15_kailh/pat1.kicad_sym D  hardware/nRF54L15_kailh/pat2.kicad_mod D  hardware/nRF54L15_kailh/pat3.kicad_mod D  hardware/nRF54L15_kailh/pat4.kicad_mod D  hardware/nRF54L15_kailh/pat5.kicad_mod D  hardware/nRF54L15_kailh/pcb/pcb-Edge_Cuts.dxf D  hardware/nRF54L15_kailh/pcb/pcb-F_Fab.dxf D  hardware/nRF54L15_kailh/pcb/pcb-User_3.dxf D  hardware/nRF54L15_kailh/pcb/pcb-User_5.dxf D  hardware/nRF54L15_kailh/pcb/pcb-User_6.dxf M  hardware/nRF54L15_kailh/placefp.py M  hardware/nRF54L15_kailh/swplate/swplate.kicad_pcb M  hardware/nRF54L15_kailh/swplate/swplate.kicad_prl M  hardware/nRF54L15_kailh/swplate/swplate.kicad_sch A  hardware/nRF54L15_kailh/test.py R  hardware/nRF54L15_kailh/tmr-footprints/DowelHole_2.9mm_M3_powdercoat.kicad_mod -> hardware/nRF54L15_kailh/tmr-footprints/DowelHole_2.8mm_M3_powdercoat.kicad_mod R  hardware/nRF54L15_kailh/tmr-footprints/DowelHole_3.0mm_M3_powdercoat.kicad_mod -> hardware/nRF54L15_kailh/tmr-footprints/PilotHole_2.05mm_M2.5_tap.kicad_mod A  hardware/nRF54L15_kailh/tmr-footprints/RivetClearanceHole_1.5mm.kicad_mod A  hardware/nRF54L15_kailh/tmr-footprints/RivetInterferenceHole_1.3mm_drill_to_1.35mm.kicad_mod M  hardware/nRF54L15_kailh/tmr-footprints/Switch_Cutout_dummy.kicad_mod D  hardware/nRF54L15_kailh/tmr-footprints/pat1.kicad_mod M  hardware/nRF54L15_kailh/topcase/topcase.kicad_pcb M  hardware/nRF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
Parts:
- H16: footprint tmr-lib:MountingHole_2.7mm_M2.5 -> tmr-lib:DowelHole_3.1mm_M3_powdercoat
- Hd1: footprint tmr-lib:DowelHole_3.2mm_M3_powdercoat -> tmr-lib:DowelHole_3.1mm_M3_powdercoat
Changed lines of the file:
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@@
 		)
 	)
-	(footprint "tmr-lib:DowelHole_3.2mm_M3_powdercoat"
+	(footprint "tmr-lib:DowelHole_3.1mm_M3_powdercoat"
 		(layer "F.Cu")
 		(at 4.55 -4.45)
@@
 		(pad "" np_thru_hole circle
 			(at 0 0)
-			(size 3.2 3.2)
-			(drill 3.2)
+			(size 3.1 3.1)
+			(drill 3.1)
 			(layers "*.Cu" "*.Mask")
 		)
@@
 		(embedded_fonts no)
 	)
-	(footprint "tmr-lib:MountingHole_2.7mm_M2.5"
+	(footprint "tmr-lib:DowelHole_3.1mm_M3_powdercoat"
 		(layer "F.Cu")
 		(at 286.75 172.5)
-		(descr "Mounting Hole 2.7mm, M2.5, no annular, generated by kicad-footprint-generator mountinghole.py")
-		(tags "mountinghole M2.5")
+		(descr "Mounting Hole 2.2mm, no annular, M2")
+		(tags "mounting hole 2.2mm no annular m2")
 		(property "Reference" "H16"
-			(at 0 -3.65 0)
-			(layer "F.SilkS")
+			(at 0 -3.2 0)
+			(layer "F.Fab")
 			(effects
 				(font
@@
 		)
 		(property "Value" "MountingHole"
-			(at 0 3.65 0)
+			(at 0 3.2 0)
 			(layer "F.Fab")
 			(effects
@@
 		(fp_circle
 			(center 0 0)
-			(end 2.7 0)
+			(end 2.2 0)
 			(stroke
 				(width 0.15)
@@
 		(fp_circle
 			(center 0 0)
-			(end 4.25 0)
+			(end 2.45 0)
 			(stroke
 				(width 0.05)
@@
 		(pad "" np_thru_hole circle
 			(at 0 0)
-			(size 2.7 2.7)
-			(drill 2.7)
+			(size 3.1 3.1)
+			(drill 3.1)
 			(layers "*.Cu" "*.Mask")
 		)
