File: hardware/nRF54L15_kailh/swplate/swplate.kicad_sch (KiCad schematic)
At the start: 102 parts

Commit message: A  hardware/nRF54L15_kailh/.gitignore M  hardware/nRF54L15_kailh/border.py A  hardware/nRF54L15_kailh/botcase/botcase-Edge_Cuts.dxf A  hardware/nRF54L15_kailh/botcase/botcase-Edge_Cuts.gm1 A  hardware/nRF54L15_kailh/botcase/botcase-Edge_Cuts.svg A  hardware/nRF54L15_kailh/botcase/botcase.kicad_pcb A  hardware/nRF54L15_kailh/botcase/botcase.kicad_prl A  hardware/nRF54L15_kailh/botcase/botcase.kicad_pro A  hardware/nRF54L15_kailh/botcase/botcase.kicad_sch A  hardware/nRF54L15_kailh/botcase/fp-lib-table A  hardware/nRF54L15_kailh/botcase/sym-lib-table A  hardware/nRF54L15_kailh/kerf.py D  hardware/nRF54L15_kailh/pat1.kicad_mod D  hardware/nRF54L15_kailh/pat1.kicad_sym D  hardware/nRF54L15_kailh/pat2.kicad_mod D  hardware/nRF54L15_kailh/pat3.kicad_mod D  hardware/nRF54L15_kailh/pat4.kicad_mod D  hardware/nRF54L15_kailh/pat5.kicad_mod D  hardware/nRF54L15_kailh/pcb/pcb-Edge_Cuts.dxf D  hardware/nRF54L15_kailh/pcb/pcb-F_Fab.dxf D  hardware/nRF54L15_kailh/pcb/pcb-User_3.dxf D  hardware/nRF54L15_kailh/pcb/pcb-User_5.dxf D  hardware/nRF54L15_kailh/pcb/pcb-User_6.dxf M  hardware/nRF54L15_kailh/placefp.py M  hardware/nRF54L15_kailh/swplate/swplate.kicad_pcb M  hardware/nRF54L15_kailh/swplate/swplate.kicad_prl M  hardware/nRF54L15_kailh/swplate/swplate.kicad_sch A  hardware/nRF54L15_kailh/test.py R  hardware/nRF54L15_kailh/tmr-footprints/DowelHole_2.9mm_M3_powdercoat.kicad_mod -> hardware/nRF54L15_kailh/tmr-footprints/DowelHole_2.8mm_M3_powdercoat.kicad_mod R  hardware/nRF54L15_kailh/tmr-footprints/DowelHole_3.0mm_M3_powdercoat.kicad_mod -> hardware/nRF54L15_kailh/tmr-footprints/PilotHole_2.05mm_M2.5_tap.kicad_mod A  hardware/nRF54L15_kailh/tmr-footprints/RivetClearanceHole_1.5mm.kicad_mod A  hardware/nRF54L15_kailh/tmr-footprints/RivetInterferenceHole_1.3mm_drill_to_1.35mm.kicad_mod M  hardware/nRF54L15_kailh/tmr-footprints/Switch_Cutout_dummy.kicad_mod D  hardware/nRF54L15_kailh/tmr-footprints/pat1.kicad_mod M  hardware/nRF54L15_kailh/topcase/topcase.kicad_pcb M  hardware/nRF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
Parts:
- H16: footprint tmr-lib:MountingHole_2.7mm_M2.5 -> tmr-lib:DowelHole_3.1mm_M3_powdercoat
- Hd1: footprint tmr-lib:DowelHole_3.2mm_M3_powdercoat -> tmr-lib:DowelHole_3.1mm_M3_powdercoat
Changed lines of the file:
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@@
 			)
 		)
-		(property "Footprint" "tmr-lib:MountingHole_2.7mm_M2.5"
+		(property "Footprint" "tmr-lib:DowelHole_3.1mm_M3_powdercoat"
 			(at 110.49 185.42 0)
 			(effects
@@
 			)
 		)
-		(property "Footprint" "tmr-lib:DowelHole_3.2mm_M3_powdercoat"
+		(property "Footprint" "tmr-lib:DowelHole_3.1mm_M3_powdercoat"
 			(at 163.83 151.13 0)
 			(effects
