File: hardware/nRF54L15_kailh/topcase/topcase.kicad_pcb (KiCad board)
At the start: 2 copper layers, 328.5 x 195.5 mm, 88 parts

Commit message: A  hardware/nRF54L15_kailh/.gitignore M  hardware/nRF54L15_kailh/border.py A  hardware/nRF54L15_kailh/botcase/botcase-Edge_Cuts.dxf A  hardware/nRF54L15_kailh/botcase/botcase-Edge_Cuts.gm1 A  hardware/nRF54L15_kailh/botcase/botcase-Edge_Cuts.svg A  hardware/nRF54L15_kailh/botcase/botcase.kicad_pcb A  hardware/nRF54L15_kailh/botcase/botcase.kicad_prl A  hardware/nRF54L15_kailh/botcase/botcase.kicad_pro A  hardware/nRF54L15_kailh/botcase/botcase.kicad_sch A  hardware/nRF54L15_kailh/botcase/fp-lib-table A  hardware/nRF54L15_kailh/botcase/sym-lib-table A  hardware/nRF54L15_kailh/kerf.py D  hardware/nRF54L15_kailh/pat1.kicad_mod D  hardware/nRF54L15_kailh/pat1.kicad_sym D  hardware/nRF54L15_kailh/pat2.kicad_mod D  hardware/nRF54L15_kailh/pat3.kicad_mod D  hardware/nRF54L15_kailh/pat4.kicad_mod D  hardware/nRF54L15_kailh/pat5.kicad_mod D  hardware/nRF54L15_kailh/pcb/pcb-Edge_Cuts.dxf D  hardware/nRF54L15_kailh/pcb/pcb-F_Fab.dxf D  hardware/nRF54L15_kailh/pcb/pcb-User_3.dxf D  hardware/nRF54L15_kailh/pcb/pcb-User_5.dxf D  hardware/nRF54L15_kailh/pcb/pcb-User_6.dxf M  hardware/nRF54L15_kailh/placefp.py M  hardware/nRF54L15_kailh/swplate/swplate.kicad_pcb M  hardware/nRF54L15_kailh/swplate/swplate.kicad_prl M  hardware/nRF54L15_kailh/swplate/swplate.kicad_sch A  hardware/nRF54L15_kailh/test.py R  hardware/nRF54L15_kailh/tmr-footprints/DowelHole_2.9mm_M3_powdercoat.kicad_mod -> hardware/nRF54L15_kailh/tmr-footprints/DowelHole_2.8mm_M3_powdercoat.kicad_mod R  hardware/nRF54L15_kailh/tmr-footprints/DowelHole_3.0mm_M3_powdercoat.kicad_mod -> hardware/nRF54L15_kailh/tmr-footprints/PilotHole_2.05mm_M2.5_tap.kicad_mod A  hardware/nRF54L15_kailh/tmr-footprints/RivetClearanceHole_1.5mm.kicad_mod A  hardware/nRF54L15_kailh/tmr-footprints/RivetInterferenceHole_1.3mm_drill_to_1.35mm.kicad_mod M  hardware/nRF54L15_kailh/tmr-footprints/Switch_Cutout_dummy.kicad_mod D  hardware/nRF54L15_kailh/tmr-footprints/pat1.kicad_mod M  hardware/nRF54L15_kailh/topcase/topcase.kicad_pcb M  hardware/nRF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
Parts:
- added Hd1: DowelHole, tmr-lib:DowelHole_2.8mm_M3_powdercoat, F.Cu at (4.55, -4.45)
- added Hd2: DowelHole, tmr-lib:DowelHole_2.8mm_M3_powdercoat, F.Cu at (262.0, 72.0)
- moved H16 326.1 mm to (286.8, 172.5)
- moved H13 318.0 mm to (286.8, 123.5)
- moved H15 258.0 mm to (209.8, 172.5)
- moved H14 244.3 mm to (209.8, 131.0)
- moved H11 149.4 mm to (65.8, 172.5)
- moved H10 124.2 mm to (65.8, 131.0)
- moved H12 112.0 mm to (-6.25, 172.5)
- moved H9 35.5 mm to (-6.25, 123.5)
- moved H1 6.45 mm to (3.00, 2.25)
- moved H4 2.50 mm to (300.0, -4.00)
- moved H7 0.25 mm to (181.2, 102.2)
- moved H5 0.05 mm to (-9.70, 71.0)
Other:
- board size 328.5 x 195.5 mm -> 328.5 x 199 mm
